Commit message: feat(gripper): isaac 后端——桥扩展 gripper articulation 读写 + isaac_gripper_action 中转 + ur5_isaac xacro
Task 5 of 6 (gripper-integration). Isaac Sim 后端 gripper:

- ur5_isaac.urdf.xacro: include gripper_macro + <xacro:lebai_gripper> +
  tool0_to_gripper_base fixed joint（mirror Task 1；不动 isaac ros2_control）.
- isaac_gripper_action.py: 暴露 control_msgs/GripperCommand action
  (lebai_gripper_controller/gripper_cmd)，goal→/isaac_gripper_joint_commands，
  读 /isaac_gripper_joint_states 判到位。MultiThreadedExecutor +
  ReentrantCallbackGroup（execute 长轮询期间订阅回调仍并发 dispatch）。
  修了 brief 骨架的 bug：重复 import、dead if-False 分支、
  goal.command.position→goal_handle.request.position、f-string logging.
- setup.py: entry_point isaac_gripper_action.
- sim_isaac.launch.py: 起 isaac_gripper_action Node.
- ur5_isaac_bridge.py: OmniGraph ActionGraph 追加 gripper articulation 读写
  (4 G-suffixed nodes / 18 connections / 4 SET_VALUES)，mirror 现有 UR5 graph。
  新增 --gripper_prim arg (default /World/gripper_abs_stl/Geometry，经 USD
  introspection 验证 ~/Desktop/scene.usd 的 ArticulationRootAPI 位置)。gripper
  驱动关节名 gripper_r_joint1 与 URDF 一致，无需映射。
- introspect_gripper.py: USD 探查脚本（记录 prim/joint 验证方式）。

Verified (offline): colcon build OK；xacro 解析含 gripper (gripper_base_link x7)；
ros2 action list 显示 /lebai_gripper_controller/gripper_cmd (1 server)；
py_compile OK。Live isaac verify deferred (heavy).

File: src/ur5_bringup/urdf/ur5_isaac.urdf.xacro (robot description, xacro)
@@ -41,4 +41,11 @@
   <!-- ===== 1) UR kinematic chain: links + joints ONLY (no default ros2_control) ===== -->
   <xacro:include filename="$(find ur_description)/urdf/ur_macro.xacro"/>
+  <!-- Lebai gripper macro (lebai_lm3_support, in-tree submodule) — mirrors Task 1
+       (ur5_with_gripper.urdf.xacro). Adds the gripper links/joints to the kinematic
+       chain so MoveIt's gripper group + the isaac bridge's gripper articulation
+       share the same URDF description. The isaac ros2_control macro below does NOT
+       cover the gripper (it only emits a <ros2_control> for the 6 arm joints); the
+       gripper is driven out-of-band via the isaac_gripper_action bridge node. -->
+  <xacro:include filename="$(find lebai_lm3_support)/urdf/gripper_macro.xacro"/>
   <xacro:ur_robot
     name="$(arg name)"
@@ -57,4 +64,13 @@
     <origin xyz="0 0 0" rpy="0 0 0"/>
   </xacro:ur_robot>
+  <!-- Lebai gripper: prefix mirrors the arm's tf_prefix (empty by default). -->
+  <xacro:lebai_gripper prefix="$(arg tf_prefix)"/>
+  <!-- Mount the gripper to the arm's tool0 (LM3 范式：identity origin；
+       若物理有转接件 offset，verify 时调). Mirrors Task 1. -->
+  <joint name="tool0_to_gripper_base" type="fixed">
+    <parent link="$(arg tf_prefix)tool0"/>
+    <child link="$(arg tf_prefix)gripper_base_link"/>
+    <origin xyz="0 0 0" rpy="0 0 0"/>
+  </joint>
   <!-- ===== 2) isaac ros2_control (TopicBasedSystem) ===== -->
   <xacro:include filename="$(find ur5_bringup)/urdf/ur5_isaac.ros2_control.xacro"/>
