Commit message: fix(urdf/real): ur5_with_gripper xacro 补全驱动参数透传（漏 arg 致 ur_ros2_control_node 拿占位符 to_be_filled 启动即 abort，真机首跑实测）；Dockerfile 补 lebai_lm3_support/lebai_resources/orbbec_description（exec_depend 不进 packages-up-to 的连环坑）

File: src/ur5_bringup/urdf/ur5_with_gripper.urdf.xacro (robot description, xacro)
@@ -14,15 +14,73 @@
   <xacro:arg name="safety_k_position" default="20"/>
   <xacro:arg name="prefix" default=""/>
+  <!-- ros2_control / 驱动参数（对齐上游 ur.urdf.xacro；real 后端必传，isaac/mock 用默认值）。
+       ⚠ 曾经的坑（2026-10-10 真机首跑）：fork 时漏了这组 arg，ur_control.launch.py 传入的
+       script_filename/RTDE recipe 落不进 <ros2_control> 参数 → 硬件接口拿到占位符
+       'to_be_filled_by_ur_robot_driver' → ur_ros2_control_node 启动即 abort(-6)。 -->
+  <xacro:arg name="name" default="ur"/>
+  <xacro:arg name="transmission_hw_interface" default=""/>
+  <xacro:arg name="headless_mode" default="false"/>
+  <xacro:arg name="robot_ip" default="0.0.0.0"/>
+  <xacro:arg name="script_filename" default=""/>
+  <xacro:arg name="output_recipe_filename" default=""/>
+  <xacro:arg name="input_recipe_filename" default=""/>
+  <xacro:arg name="reverse_ip" default="0.0.0.0"/>
+  <xacro:arg name="script_command_port" default="50004"/>
+  <xacro:arg name="reverse_port" default="50001"/>
+  <xacro:arg name="script_sender_port" default="50002"/>
+  <xacro:arg name="trajectory_port" default="50003"/>
+  <xacro:arg name="use_tool_communication" default="false"/>
+  <xacro:arg name="tool_voltage" default="0"/>
+  <xacro:arg name="tool_parity" default="0"/>
+  <xacro:arg name="tool_baud_rate" default="115200"/>
+  <xacro:arg name="tool_stop_bits" default="1"/>
+  <xacro:arg name="tool_rx_idle_chars" default="1.5"/>
+  <xacro:arg name="tool_tx_idle_chars" default="3.5"/>
+  <xacro:arg name="tool_device_name" default="/tmp/ttyUR"/>
+  <xacro:arg name="tool_tcp_port" default="54321"/>
+  <xacro:arg name="use_fake_hardware" default="false"/>
+  <xacro:arg name="fake_sensor_commands" default="false"/>
+  <xacro:arg name="sim_gazebo" default="false"/>
+  <xacro:arg name="sim_ignition" default="false"/>
+  <xacro:arg name="simulation_controllers" default=""/>
+  <xacro:arg name="initial_positions_file" default="$(find ur_description)/config/initial_positions.yaml"/>
+  <xacro:property name="initial_positions_file" value="$(arg initial_positions_file)"/>
   <!-- World link for base attachment -->
   <link name="world"/>
-  <!-- UR5 arm macro: actual macro name is ur_robot, uses tf_prefix & parent + *origin block -->
-  <xacro:ur_robot name="ur" tf_prefix="$(arg prefix)" parent="world"
+  <!-- UR5 arm macro: actual macro name is ur_robot, uses tf_prefix & parent + *origin block。
+       ros2_control/驱动参数全量透传（对齐上游 ur.urdf.xacro 的调用）。 -->
+  <xacro:ur_robot name="$(arg name)" tf_prefix="$(arg prefix)" parent="world"
             joint_limits_parameters_file="$(arg joint_limit_params)"
             kinematics_parameters_file="$(arg kinematics_params)"
             physical_parameters_file="$(arg physical_params)"
             visual_parameters_file="$(arg visual_params)"
+            transmission_hw_interface="$(arg transmission_hw_interface)"
             safety_limits="$(arg safety_limits)"
             safety_pos_margin="$(arg safety_pos_margin)"
-            safety_k_position="$(arg safety_k_position)">
+            safety_k_position="$(arg safety_k_position)"
+            use_fake_hardware="$(arg use_fake_hardware)"
+            fake_sensor_commands="$(arg fake_sensor_commands)"
+            sim_gazebo="$(arg sim_gazebo)"
+            sim_ignition="$(arg sim_ignition)"
+            headless_mode="$(arg headless_mode)"
+            initial_positions="${xacro.load_yaml(initial_positions_file)}"
+            use_tool_communication="$(arg use_tool_communication)"
+            tool_voltage="$(arg tool_voltage)"
+            tool_parity="$(arg tool_parity)"
+            tool_baud_rate="$(arg tool_baud_rate)"
+            tool_stop_bits="$(arg tool_stop_bits)"
+            tool_rx_idle_chars="$(arg tool_rx_idle_chars)"
+            tool_tx_idle_chars="$(arg tool_tx_idle_chars)"
+            tool_device_name="$(arg tool_device_name)"
+            tool_tcp_port="$(arg tool_tcp_port)"
+            robot_ip="$(arg robot_ip)"
+            script_filename="$(arg script_filename)"
+            output_recipe_filename="$(arg output_recipe_filename)"
+            input_recipe_filename="$(arg input_recipe_filename)"
+            reverse_ip="$(arg reverse_ip)"
+            script_command_port="$(arg script_command_port)"
+            reverse_port="$(arg reverse_port)"
+            script_sender_port="$(arg script_sender_port)"
+            trajectory_port="$(arg trajectory_port)">
     <origin xyz="0 0 0" rpy="0 0 0"/>
   </xacro:ur_robot>
