Commit message: fix(isaac-gripper): 焊进 UR5 articulation + 夹爪端到端可用 + RViz 球到 gripper_tip
isaac 后端夹爪 plan/execute/开合全通，RViz 目标交互球落到夹爪 tip。一路修的坑：

- scene (~/Desktop/scene.usd, fix_gripper_anchor.py): 删夹爪 NewtonArticulationRootAPI
  + 禁用钉地的 root_joint → 夹爪经 AssemblerFixedJoint 并入 /World/ur5/root_joint
  （之前夹爪既钉地又焊手臂 → 手臂被锁、execute 不动）
- bridge (ur5_isaac_bridge.py): 夹爪 OmniGraph 改指合并根 /World/ur5/root_joint
  （与 arm 同根；两个 ArticulationController 按 jointNames 不互踩）
- ros2_control (ur5_isaac.ros2_control.xacro): 夹爪关节不放进来——state-only 会让
  TopicBasedSystem 发畸形的 /isaac_joint_commands（name/position 长度不匹配 → 桥不驱动）
- isaac_gripper_action.py: 把 gripper_r_joint1 转发到 /joint_states（绕开 ros2_control）
- moveit.launch.py: lebai_gripper_controller 加进 controller_names + action_ns=gripper_cmd
  （原 action_ns 全路径 → MoveIt 拼成双前缀 .../lebai_gripper_controller/gripper_cmd）
- URDF (ur5_with_gripper.urdf.xacro): 加固定 TCP 链 gripper_tip_tcp（z=0.17127）
- SRDF (ur5_with_gripper.srdf.xacro): fork ur_manipulator chain tip → gripper_tip_tcp
  （内联 ur_macro.srdf.xacro 的 group/states/disable_collisions），end_effector 重指；
  arm 仍 6-DOF，joint_trajectory_controller 不变

工具：weld_gripper.py / fix_gripper_anchor.py / introspect_{assembly,mount_geometry,gripper_offset}.py

File: src/ur5_bringup/srdf/ur5_with_gripper.srdf.xacro (robot description, xacro)
@@ -3,17 +3,59 @@
   <!--
     SRDF for ur5 + Lebai gripper.
-    Includes the system ur_moveit SRDF (ur_manipulator group, virtual_joint,
-    disable_collisions for the arm) and appends the Lebai gripper block.
-    Group/joint/state names mirror lebai_lm3_moveit_config/config/lebai_lm3.srdf;
-    disable_collisions copied verbatim from that file (gripper-internal pairs only —
-    arm-internal pairs come from the included ur.srdf.xacro).
+    ur_manipulator group 是本地 fork（内联系统 ur_macro.srdf.xacro 的 group/states/arm
+    disable_collisions），唯一改动：chain tip = gripper_tip_tcp（URDF 里加的固定 TCP 帧），
+    让 RViz 目标交互球 / IK 目标落在夹爪 tip。arm 仍 6-DOF。
+    后面是 Lebai gripper block（group/end_effector/open-closed/disable_collisions），
+    group/joint/state 名镜像 lebai_lm3_moveit_config/config/lebai_lm3.srdf。
   -->
-  <!-- system ur_moveit SRDF: ur_manipulator group + arm disable_collisions -->
-  <xacro:include filename="$(find ur_moveit_config)/srdf/ur.srdf.xacro"/>
+  <!-- ===== ur_manipulator: 本地 fork（原 <xacro:include ur.srdf.xacro/> 的 ur_srdf 宏内联）=====
+       唯一改动：chain tip 从 tool0 → gripper_tip_tcp（URDF 里加的固定 TCP 帧，与 gripper_tip 共位）。
+       这样 MoveIt 的目标交互球 / IK 目标落在夹爪 tip 而非法兰。固定 joint=0 DOF → 仍 6-DOF arm 规划，
+       joint_trajectory_controller 仍收 6 arm 关节，组名 ur_manipulator 不变（kinematics/OMPL/servo 不动）。
+       不能直接把 tip 设成 gripper_tip——会拖进 3 个 mimic revolute 关节变 9-DOF 炸控制器。 -->
+  <group name="ur_manipulator">
+    <chain base_link="base_link" tip_link="gripper_tip_tcp" />
+  </group>
+  <group_state name="home" group="ur_manipulator">
+    <joint name="elbow_joint" value="0" />
+    <joint name="shoulder_lift_joint" value="-1.5707" />
+    <joint name="shoulder_pan_joint" value="0" />
+    <joint name="wrist_1_joint" value="0" />
+    <joint name="wrist_2_joint" value="0" />
+    <joint name="wrist_3_joint" value="0" />
+  </group_state>
+  <group_state name="up" group="ur_manipulator">
+    <joint name="elbow_joint" value="0" />
+    <joint name="shoulder_lift_joint" value="-1.5707" />
+    <joint name="shoulder_pan_joint" value="0" />
+    <joint name="wrist_1_joint" value="-1.5707" />
+    <joint name="wrist_2_joint" value="0" />
+    <joint name="wrist_3_joint" value="0" />
+  </group_state>
+  <group_state name="test_configuration" group="ur_manipulator">
+    <joint name="elbow_joint" value="1.4" />
+    <joint name="shoulder_lift_joint" value="-1.62" />
+    <joint name="shoulder_pan_joint" value="1.54" />
+    <joint name="wrist_1_joint" value="-1.2" />
+    <joint name="wrist_2_joint" value="-1.6" />
+    <joint name="wrist_3_joint" value="-0.11" />
+  </group_state>
+  <!-- arm-internal disable_collisions（照搬 ur_macro.srdf.xacro）-->
+  <disable_collisions link1="base_link" link2="base_link_inertia" reason="Adjacent" />
+  <disable_collisions link1="base_link_inertia" link2="shoulder_link" reason="Adjacent" />
+  <disable_collisions link1="tool0" link2="wrist_1_link" reason="Never" />
+  <disable_collisions link1="tool0" link2="wrist_2_link" reason="Never" />
+  <disable_collisions link1="tool0" link2="wrist_3_link" reason="Adjacent" />
+  <disable_collisions link1="forearm_link" link2="upper_arm_link" reason="Adjacent" />
+  <disable_collisions link1="forearm_link" link2="wrist_1_link" reason="Adjacent" />
+  <disable_collisions link1="shoulder_link" link2="upper_arm_link" reason="Adjacent" />
+  <disable_collisions link1="wrist_1_link" link2="wrist_2_link" reason="Adjacent" />
+  <disable_collisions link1="wrist_1_link" link2="wrist_3_link" reason="Never" />
+  <disable_collisions link1="wrist_2_link" link2="wrist_3_link" reason="Adjacent" />
   <!-- ===== Lebai gripper (from lebai_lm3_moveit_config/config/lebai_lm3.srdf) ===== -->
   <group name="gripper">
     <joint name="gripper_r_joint1"/>
   </group>
-  <end_effector name="gripper" parent_link="tool0" group="gripper" parent_group="ur_manipulator"/>
+  <end_effector name="gripper" parent_link="gripper_tip_tcp" group="gripper" parent_group="ur_manipulator"/>
   <group_state name="open" group="gripper">
     <joint name="gripper_r_joint1" value="1.0471975512"/>

File: src/ur5_bringup/urdf/ur5_isaac.ros2_control.xacro (robot description, xacro)
@@ -85,4 +85,9 @@
         </state_interface>
       </joint>
+      <!-- NOTE: gripper_r_joint1 故意不在 ros2_control 里。之前加过 state-only 接口，
+           但 TopicBasedSystem 会把它塞进 /isaac_joint_commands 的 name 列表（却不带
+           command 值）→ name/position 长度不匹配 → 桥收到畸形消息不驱动 → 手臂不动。
+           夹爪关节状态改由独立途径发到 /joint_states（见 isaac_gripper_action /
+           relay），不经过 ros2_control。-->
     </ros2_control>
   </xacro:macro>

File: src/ur5_bringup/urdf/ur5_isaac.urdf.xacro (robot description, xacro)
@@ -71,5 +71,7 @@
     <parent link="$(arg tf_prefix)tool0"/>
     <child link="$(arg tf_prefix)gripper_base_link"/>
-    <origin xyz="0 0 0" rpy="0 0 0"/>
+    <!-- 转接环 offset：沿 tool0 Z 把夹爪 base 撑离 flange（实测场景 +0.01267m，无转角）。
+         与 ur5_with_gripper.urdf.xacro 保持一致。先按场景值试，不够再调。 -->
+    <origin xyz="0 0 0.01267" rpy="0 0 0"/>
   </joint>
   <!-- ===== 2) isaac ros2_control (TopicBasedSystem) ===== -->

File: src/ur5_bringup/urdf/ur5_with_gripper.urdf.xacro (robot description, xacro)
@@ -33,5 +33,17 @@
     <parent link="$(arg prefix)tool0"/>
     <child link="$(arg prefix)gripper_base_link"/>
-    <origin xyz="0 0 0" rpy="0 0 0"/>
+    <!-- 转接环 offset：沿 tool0 Z 把夹爪 base 撑离 flange（实测场景 gripper_base 相对
+         wrist_3 沿工具轴 +0.01267m，无转角）。先按场景值试，不够再调。 -->
+    <origin xyz="0 0 0.01267" rpy="0 0 0"/>
+  </joint>
+  <!-- 固定 TCP 帧（与 gripper_tip 共位），供 IK / RViz 目标交互球定位。
+       tool0→gripper_tip 在任意指角下为纯 Z 平移（3 个 mimic 关节净转角 θ−2θ+θ=0）：
+       mount(0.01267) + 0.1056 + 0.0265 + 0.0265 = 0.17127 m。固定 joint=0 DOF，
+       arm 规划仍 6-DOF。chain tip 指 gripper_tip_tcp 后，RViz 的目标球就落这里。 -->
+  <link name="$(arg prefix)gripper_tip_tcp"/>
+  <joint name="tool0_to_gripper_tip_tcp" type="fixed">
+    <parent link="$(arg prefix)tool0"/>
+    <child link="$(arg prefix)gripper_tip_tcp"/>
+    <origin xyz="0 0 0.17127" rpy="0 0 0"/>
   </joint>
 </robot>

Commit message: feat(isaac): 抓取栈就绪 + scene.usd 渲染修复
- P1 RViz 默认 OMPL（moveit_client planner_id PTP→""）
- P2 world→base TF 自动同步（桥读 USD base 发 tf_static；real 参数化抬升 arg）
- P3 depth 显示（gemini_2 补 camera_depth_optical_frame；fork rviz 加 Image/DepthCloud 默认不勾）
- P4 抓取（publish_object_pose 读 USD 瓶子 GT 位姿发 /grasp_target_pose；demo_grasp 订阅抓取；moveit_client 加 attach/detach）
- scene.usd: 桌面 OmniPBR 材质修复 + 相机 near clipping 1m→0.05m
- submodule OrbbecSDK: gemini_2 depth optical 补丁（ffbe4a84）

File: src/ur5_bringup/srdf/ur5_with_gripper.srdf.xacro (robot description, xacro)
@@ -88,3 +88,83 @@
   <disable_collisions link1="gripper_r_link1" link2="gripper_r_link_finger" reason="Never"/>
   <disable_collisions link1="gripper_r_link2" link2="gripper_r_link_finger" reason="Never"/>
+  <!-- ===== Orbbec 相机：camera_link + camera_botter_screw_frame vs 全部手臂/夹爪 link（刚性挂载，不做自碰撞）===== -->
+  <disable_collisions link1="camera_link" link2="base_link" reason="Never"/>
+  <disable_collisions link1="camera_link" link2="base_link_inertia" reason="Never"/>
+  <disable_collisions link1="camera_link" link2="shoulder_link" reason="Never"/>
+  <disable_collisions link1="camera_link" link2="upper_arm_link" reason="Never"/>
+  <disable_collisions link1="camera_link" link2="forearm_link" reason="Never"/>
+  <disable_collisions link1="camera_link" link2="wrist_1_link" reason="Never"/>
+  <disable_collisions link1="camera_link" link2="wrist_2_link" reason="Never"/>
+  <disable_collisions link1="camera_link" link2="wrist_3_link" reason="Never"/>
+  <disable_collisions link1="camera_link" link2="flange" reason="Never"/>
+  <disable_collisions link1="camera_link" link2="tool0" reason="Never"/>
+  <disable_collisions link1="camera_link" link2="gripper_base_link" reason="Never"/>
+  <disable_collisions link1="camera_link" link2="gripper_r_link1" reason="Never"/>
+  <disable_collisions link1="camera_link" link2="gripper_r_link2" reason="Never"/>
+  <disable_collisions link1="camera_link" link2="gripper_r_link_finger" reason="Never"/>
+  <disable_collisions link1="camera_link" link2="gripper_l_link1" reason="Never"/>
+  <disable_collisions link1="camera_link" link2="gripper_l_link2" reason="Never"/>
+  <disable_collisions link1="camera_link" link2="gripper_l_link_finger" reason="Never"/>
+  <disable_collisions link1="camera_link" link2="gripper_tip_midpoint_arm" reason="Never"/>
+  <disable_collisions link1="camera_link" link2="gripper_tip_midpoint_counterarm" reason="Never"/>
+  <disable_collisions link1="camera_link" link2="gripper_tip" reason="Never"/>
+  <disable_collisions link1="camera_link" link2="camera_flange_support" reason="Adjacent"/>
+  <disable_collisions link1="camera_botter_screw_frame" link2="base_link" reason="Never"/>
+  <disable_collisions link1="camera_botter_screw_frame" link2="shoulder_link" reason="Never"/>
+  <disable_collisions link1="camera_botter_screw_frame" link2="upper_arm_link" reason="Never"/>
+  <disable_collisions link1="camera_botter_screw_frame" link2="forearm_link" reason="Never"/>
+  <disable_collisions link1="camera_botter_screw_frame" link2="wrist_1_link" reason="Never"/>
+  <disable_collisions link1="camera_botter_screw_frame" link2="wrist_2_link" reason="Never"/>
+  <disable_collisions link1="camera_botter_screw_frame" link2="wrist_3_link" reason="Never"/>
+  <disable_collisions link1="camera_botter_screw_frame" link2="flange" reason="Never"/>
+  <disable_collisions link1="camera_botter_screw_frame" link2="tool0" reason="Never"/>
+  <disable_collisions link1="camera_botter_screw_frame" link2="gripper_base_link" reason="Never"/>
+  <disable_collisions link1="camera_botter_screw_frame" link2="gripper_r_link1" reason="Never"/>
+  <disable_collisions link1="camera_botter_screw_frame" link2="gripper_l_link1" reason="Never"/>
+  <disable_collisions link1="camera_botter_screw_frame" link2="camera_flange_support" reason="Adjacent"/>
+  <!-- 相机内部（相邻 link，不做碰撞）-->
+  <disable_collisions link1="camera_link" link2="camera_botter_screw_frame" reason="Adjacent"/>
+  <disable_collisions link1="camera_link" link2="camera_depth_frame" reason="Adjacent"/>
+  <disable_collisions link1="camera_link" link2="camera_left_ir_frame" reason="Adjacent"/>
+  <disable_collisions link1="camera_depth_frame" link2="camera_color_frame" reason="Adjacent"/>
+  <disable_collisions link1="camera_depth_frame" link2="camera_right_ir_frame" reason="Adjacent"/>
+  <disable_collisions link1="camera_color_frame" link2="camera_color_optical_frame" reason="Adjacent"/>
+  <disable_collisions link1="camera_right_ir_frame" link2="camera_right_ir_optical_frame" reason="Adjacent"/>
+  <disable_collisions link1="camera_left_ir_frame" link2="camera_left_ir_optical_frame" reason="Adjacent"/>
+  <!-- 相机内部非相邻对（刚性整体，全部不自碰撞）-->
+  <disable_collisions link1="camera_link" link2="camera_color_frame" reason="Never"/>
+  <disable_collisions link1="camera_link" link2="camera_color_optical_frame" reason="Never"/>
+  <disable_collisions link1="camera_link" link2="camera_right_ir_frame" reason="Never"/>
+  <disable_collisions link1="camera_link" link2="camera_right_ir_optical_frame" reason="Never"/>
+  <disable_collisions link1="camera_link" link2="camera_left_ir_optical_frame" reason="Never"/>
+  <disable_collisions link1="camera_botter_screw_frame" link2="camera_depth_frame" reason="Never"/>
+  <disable_collisions link1="camera_botter_screw_frame" link2="camera_color_frame" reason="Never"/>
+  <disable_collisions link1="camera_botter_screw_frame" link2="camera_color_optical_frame" reason="Never"/>
+  <disable_collisions link1="camera_botter_screw_frame" link2="camera_right_ir_frame" reason="Never"/>
+  <disable_collisions link1="camera_botter_screw_frame" link2="camera_right_ir_optical_frame" reason="Never"/>
+  <disable_collisions link1="camera_botter_screw_frame" link2="camera_left_ir_frame" reason="Never"/>
+  <disable_collisions link1="camera_botter_screw_frame" link2="camera_left_ir_optical_frame" reason="Never"/>
+  <disable_collisions link1="camera_depth_frame" link2="camera_color_optical_frame" reason="Never"/>
+  <disable_collisions link1="camera_depth_frame" link2="camera_right_ir_optical_frame" reason="Never"/>
+  <disable_collisions link1="camera_depth_frame" link2="camera_left_ir_optical_frame" reason="Never"/>
+  <disable_collisions link1="camera_depth_frame" link2="camera_left_ir_frame" reason="Never"/>
+  <disable_collisions link1="camera_depth_frame" link2="camera_botter_screw_frame" reason="Never"/>
+  <disable_collisions link1="camera_color_frame" link2="camera_right_ir_frame" reason="Never"/>
+  <disable_collisions link1="camera_color_frame" link2="camera_right_ir_optical_frame" reason="Never"/>
+  <disable_collisions link1="camera_color_frame" link2="camera_left_ir_frame" reason="Never"/>
+  <disable_collisions link1="camera_color_frame" link2="camera_left_ir_optical_frame" reason="Never"/>
+  <disable_collisions link1="camera_color_frame" link2="camera_botter_screw_frame" reason="Never"/>
+  <disable_collisions link1="camera_right_ir_frame" link2="camera_left_ir_frame" reason="Never"/>
+  <disable_collisions link1="camera_right_ir_frame" link2="camera_left_ir_optical_frame" reason="Never"/>
+  <disable_collisions link1="camera_right_ir_frame" link2="camera_color_optical_frame" reason="Never"/>
+  <disable_collisions link1="camera_right_ir_frame" link2="camera_botter_screw_frame" reason="Never"/>
+  <disable_collisions link1="camera_right_ir_optical_frame" link2="camera_left_ir_frame" reason="Never"/>
+  <disable_collisions link1="camera_right_ir_optical_frame" link2="camera_left_ir_optical_frame" reason="Never"/>
+  <disable_collisions link1="camera_right_ir_optical_frame" link2="camera_color_optical_frame" reason="Never"/>
+  <disable_collisions link1="camera_right_ir_optical_frame" link2="camera_botter_screw_frame" reason="Never"/>
+  <disable_collisions link1="camera_left_ir_frame" link2="camera_color_optical_frame" reason="Never"/>
+  <disable_collisions link1="camera_left_ir_frame" link2="camera_botter_screw_frame" reason="Never"/>
+  <disable_collisions link1="camera_left_ir_optical_frame" link2="camera_color_optical_frame" reason="Never"/>
+  <disable_collisions link1="camera_left_ir_optical_frame" link2="camera_botter_screw_frame" reason="Never"/>
+  <disable_collisions link1="camera_color_optical_frame" link2="camera_botter_screw_frame" reason="Never"/>
 </robot>

File: src/ur5_bringup/urdf/ur5_isaac.urdf.xacro (robot description, xacro)
@@ -75,4 +75,27 @@
     <origin xyz="0 0 0.01267" rpy="0 0 0"/>
   </joint>
+  <!-- Orbbec Gemini 2 相机（官方 gemini_2.urdf.xacro，eye-in-hand 挂 flange）。
+       mount 位姿 = USD 实测（orbbec_gemini_2 相对 flange）：xyz=(0,0,0), rpy=(0,0,-90°)。
+       带 mesh + REP-103 光学帧。与 ur5_with_gripper.urdf.xacro 一致。-->
+  <xacro:include filename="$(find orbbec_description)/urdf/gemini_2.urdf.xacro"/>
+  <joint name="flange_to_camera_link" type="fixed">
+    <parent link="$(arg tf_prefix)flange"/>
+    <child link="camera_link"/>
+    <origin xyz="0.026 0.028 0.0579" rpy="0 0 0"/>
+  </joint>
+  <!-- cameraURflangeSupport 转接环（visual only；STL mm 制 scale 0.001）-->
+  <link name="camera_flange_support">
+    <visual>
+      <geometry>
+        <mesh filename="package://ur5_bringup/meshes/realsenseURflangeSupport.stl" scale="0.001 0.001 0.001"/>
+      </geometry>
+      <material name="flange_support_gray"><color rgba="0.5 0.5 0.5 1"/></material>
+    </visual>
+  </link>
+  <joint name="flange_to_camera_flange_support" type="fixed">
+    <parent link="$(arg tf_prefix)flange"/>
+    <child link="camera_flange_support"/>
+    <origin xyz="0 0 0" rpy="0 0 1.5708"/>
+  </joint>
   <!-- ===== 2) isaac ros2_control (TopicBasedSystem) ===== -->
   <xacro:include filename="$(find ur5_bringup)/urdf/ur5_isaac.ros2_control.xacro"/>

File: src/ur5_bringup/urdf/ur5_with_gripper.urdf.xacro (robot description, xacro)
@@ -47,3 +47,26 @@
     <origin xyz="0 0 0.17127" rpy="0 0 0"/>
   </joint>
+  <!-- Orbbec Gemini 2 相机（官方 orbbec_description/urdf/gemini_2.urdf.xacro，eye-in-hand）。
+       mount 位姿 = USD 实测（orbbec_gemini_2 相对 flange）：xyz=(0,0,0), rpy=(0,0,-90°)。
+       带 mesh + REP-103 光学帧。M7 手眼标定再精修。-->
+  <xacro:include filename="$(find orbbec_description)/urdf/gemini_2.urdf.xacro"/>
+  <joint name="flange_to_camera_link" type="fixed">
+    <parent link="$(arg prefix)flange"/>
+    <child link="camera_link"/>
+    <origin xyz="0.026 0.028 0.0579" rpy="0 0 0"/>
+  </joint>
+  <!-- cameraURflangeSupport 转接环（visual only；STL 原始 mm 制，scale 0.001 转 m）-->
+  <link name="camera_flange_support">
+    <visual>
+      <geometry>
+        <mesh filename="package://ur5_bringup/meshes/realsenseURflangeSupport.stl" scale="0.001 0.001 0.001"/>
+      </geometry>
+      <material name="flange_support_gray"><color rgba="0.5 0.5 0.5 1"/></material>
+    </visual>
+  </link>
+  <joint name="flange_to_camera_flange_support" type="fixed">
+    <parent link="$(arg prefix)flange"/>
+    <child link="camera_flange_support"/>
+    <origin xyz="0 0 0" rpy="0 0 1.5708"/>
+  </joint>
 </robot>
