Commit message: fix(srdf): robot 名对齐 URDF + 相机子帧自碰撞对
- name: ur5 → ur5_with_gripper（与 moveit.launch.py 的 URDF 一致；
  不一致时 move_group 报 Semantic description is not specified for
  the same robot，一个 group 都不加载，/compute_ik 全废）
- 8 个相机子帧(color/depth/ir+optical) vs 全部手臂/夹爪 link 的
  disable_collisions×168：不加则 forearm↔camera 假自碰撞让 OMPL
  拒合法路径(-2 INVALID_MOTION_PLAN)

File: src/ur5_bringup/srdf/ur5_with_gripper.srdf.xacro (robot description, xacro)
@@ -1,4 +1,4 @@
 <?xml version="1.0"?>
-<robot xmlns:xacro="http://ros.org/wiki/xacro" name="ur5">
+<robot xmlns:xacro="http://ros.org/wiki/xacro" name="ur5_with_gripper">
   <!--
     SRDF for ur5 + Lebai gripper.
@@ -19,5 +19,5 @@
   <group_state name="home" group="ur_manipulator">
     <joint name="elbow_joint" value="0" />
-    <joint name="shoulder_lift_joint" value="-1.5707" />
+    <joint name="shoulder_lift_joint" value="-0.7854" />
     <joint name="shoulder_pan_joint" value="0" />
     <joint name="wrist_1_joint" value="0" />
@@ -27,5 +27,5 @@
   <group_state name="up" group="ur_manipulator">
     <joint name="elbow_joint" value="0" />
-    <joint name="shoulder_lift_joint" value="-1.5707" />
+    <joint name="shoulder_lift_joint" value="-0.7854" />
     <joint name="shoulder_pan_joint" value="0" />
     <joint name="wrist_1_joint" value="-1.5707" />
@@ -168,3 +168,174 @@
   <disable_collisions link1="camera_left_ir_optical_frame" link2="camera_botter_screw_frame" reason="Never"/>
   <disable_collisions link1="camera_color_optical_frame" link2="camera_botter_screw_frame" reason="Never"/>
+  <!-- ===== 相机 8 个子帧(color/depth/ir + 各自 optical) vs 全部手臂/夹爪 link：
+       刚性挂载在 flange，整组不做自碰撞。之前漏配 → forearm vs camera_left_ir_optical_frame
+       等假自碰撞，让 OMPL 判路径 invalid(-2)，运动时灵时不灵。补全。===== -->
+  <disable_collisions link1="camera_color_frame" link2="base_link" reason="Never"/>
+  <disable_collisions link1="camera_color_frame" link2="base_link_inertia" reason="Never"/>
+  <disable_collisions link1="camera_color_frame" link2="shoulder_link" reason="Never"/>
+  <disable_collisions link1="camera_color_frame" link2="upper_arm_link" reason="Never"/>
+  <disable_collisions link1="camera_color_frame" link2="forearm_link" reason="Never"/>
+  <disable_collisions link1="camera_color_frame" link2="wrist_1_link" reason="Never"/>
+  <disable_collisions link1="camera_color_frame" link2="wrist_2_link" reason="Never"/>
+  <disable_collisions link1="camera_color_frame" link2="wrist_3_link" reason="Never"/>
+  <disable_collisions link1="camera_color_frame" link2="flange" reason="Never"/>
+  <disable_collisions link1="camera_color_frame" link2="tool0" reason="Never"/>
+  <disable_collisions link1="camera_color_frame" link2="gripper_base_link" reason="Never"/>
+  <disable_collisions link1="camera_color_frame" link2="gripper_r_link1" reason="Never"/>
+  <disable_collisions link1="camera_color_frame" link2="gripper_r_link2" reason="Never"/>
+  <disable_collisions link1="camera_color_frame" link2="gripper_r_link_finger" reason="Never"/>
+  <disable_collisions link1="camera_color_frame" link2="gripper_l_link1" reason="Never"/>
+  <disable_collisions link1="camera_color_frame" link2="gripper_l_link2" reason="Never"/>
+  <disable_collisions link1="camera_color_frame" link2="gripper_l_link_finger" reason="Never"/>
+  <disable_collisions link1="camera_color_frame" link2="gripper_tip_midpoint_arm" reason="Never"/>
+  <disable_collisions link1="camera_color_frame" link2="gripper_tip_midpoint_counterarm" reason="Never"/>
+  <disable_collisions link1="camera_color_frame" link2="gripper_tip" reason="Never"/>
+  <disable_collisions link1="camera_color_frame" link2="camera_flange_support" reason="Never"/>
+  <disable_collisions link1="camera_color_optical_frame" link2="base_link" reason="Never"/>
+  <disable_collisions link1="camera_color_optical_frame" link2="base_link_inertia" reason="Never"/>
+  <disable_collisions link1="camera_color_optical_frame" link2="shoulder_link" reason="Never"/>
+  <disable_collisions link1="camera_color_optical_frame" link2="upper_arm_link" reason="Never"/>
+  <disable_collisions link1="camera_color_optical_frame" link2="forearm_link" reason="Never"/>
+  <disable_collisions link1="camera_color_optical_frame" link2="wrist_1_link" reason="Never"/>
+  <disable_collisions link1="camera_color_optical_frame" link2="wrist_2_link" reason="Never"/>
+  <disable_collisions link1="camera_color_optical_frame" link2="wrist_3_link" reason="Never"/>
+  <disable_collisions link1="camera_color_optical_frame" link2="flange" reason="Never"/>
+  <disable_collisions link1="camera_color_optical_frame" link2="tool0" reason="Never"/>
+  <disable_collisions link1="camera_color_optical_frame" link2="gripper_base_link" reason="Never"/>
+  <disable_collisions link1="camera_color_optical_frame" link2="gripper_r_link1" reason="Never"/>
+  <disable_collisions link1="camera_color_optical_frame" link2="gripper_r_link2" reason="Never"/>
+  <disable_collisions link1="camera_color_optical_frame" link2="gripper_r_link_finger" reason="Never"/>
+  <disable_collisions link1="camera_color_optical_frame" link2="gripper_l_link1" reason="Never"/>
+  <disable_collisions link1="camera_color_optical_frame" link2="gripper_l_link2" reason="Never"/>
+  <disable_collisions link1="camera_color_optical_frame" link2="gripper_l_link_finger" reason="Never"/>
+  <disable_collisions link1="camera_color_optical_frame" link2="gripper_tip_midpoint_arm" reason="Never"/>
+  <disable_collisions link1="camera_color_optical_frame" link2="gripper_tip_midpoint_counterarm" reason="Never"/>
+  <disable_collisions link1="camera_color_optical_frame" link2="gripper_tip" reason="Never"/>
+  <disable_collisions link1="camera_color_optical_frame" link2="camera_flange_support" reason="Never"/>
+  <disable_collisions link1="camera_depth_frame" link2="base_link" reason="Never"/>
+  <disable_collisions link1="camera_depth_frame" link2="base_link_inertia" reason="Never"/>
+  <disable_collisions link1="camera_depth_frame" link2="shoulder_link" reason="Never"/>
+  <disable_collisions link1="camera_depth_frame" link2="upper_arm_link" reason="Never"/>
+  <disable_collisions link1="camera_depth_frame" link2="forearm_link" reason="Never"/>
+  <disable_collisions link1="camera_depth_frame" link2="wrist_1_link" reason="Never"/>
+  <disable_collisions link1="camera_depth_frame" link2="wrist_2_link" reason="Never"/>
+  <disable_collisions link1="camera_depth_frame" link2="wrist_3_link" reason="Never"/>
+  <disable_collisions link1="camera_depth_frame" link2="flange" reason="Never"/>
+  <disable_collisions link1="camera_depth_frame" link2="tool0" reason="Never"/>
+  <disable_collisions link1="camera_depth_frame" link2="gripper_base_link" reason="Never"/>
+  <disable_collisions link1="camera_depth_frame" link2="gripper_r_link1" reason="Never"/>
+  <disable_collisions link1="camera_depth_frame" link2="gripper_r_link2" reason="Never"/>
+  <disable_collisions link1="camera_depth_frame" link2="gripper_r_link_finger" reason="Never"/>
+  <disable_collisions link1="camera_depth_frame" link2="gripper_l_link1" reason="Never"/>
+  <disable_collisions link1="camera_depth_frame" link2="gripper_l_link2" reason="Never"/>
+  <disable_collisions link1="camera_depth_frame" link2="gripper_l_link_finger" reason="Never"/>
+  <disable_collisions link1="camera_depth_frame" link2="gripper_tip_midpoint_arm" reason="Never"/>
+  <disable_collisions link1="camera_depth_frame" link2="gripper_tip_midpoint_counterarm" reason="Never"/>
+  <disable_collisions link1="camera_depth_frame" link2="gripper_tip" reason="Never"/>
+  <disable_collisions link1="camera_depth_frame" link2="camera_flange_support" reason="Never"/>
+  <disable_collisions link1="camera_depth_optical_frame" link2="base_link" reason="Never"/>
+  <disable_collisions link1="camera_depth_optical_frame" link2="base_link_inertia" reason="Never"/>
+  <disable_collisions link1="camera_depth_optical_frame" link2="shoulder_link" reason="Never"/>
+  <disable_collisions link1="camera_depth_optical_frame" link2="upper_arm_link" reason="Never"/>
+  <disable_collisions link1="camera_depth_optical_frame" link2="forearm_link" reason="Never"/>
+  <disable_collisions link1="camera_depth_optical_frame" link2="wrist_1_link" reason="Never"/>
+  <disable_collisions link1="camera_depth_optical_frame" link2="wrist_2_link" reason="Never"/>
+  <disable_collisions link1="camera_depth_optical_frame" link2="wrist_3_link" reason="Never"/>
+  <disable_collisions link1="camera_depth_optical_frame" link2="flange" reason="Never"/>
+  <disable_collisions link1="camera_depth_optical_frame" link2="tool0" reason="Never"/>
+  <disable_collisions link1="camera_depth_optical_frame" link2="gripper_base_link" reason="Never"/>
+  <disable_collisions link1="camera_depth_optical_frame" link2="gripper_r_link1" reason="Never"/>
+  <disable_collisions link1="camera_depth_optical_frame" link2="gripper_r_link2" reason="Never"/>
+  <disable_collisions link1="camera_depth_optical_frame" link2="gripper_r_link_finger" reason="Never"/>
+  <disable_collisions link1="camera_depth_optical_frame" link2="gripper_l_link1" reason="Never"/>
+  <disable_collisions link1="camera_depth_optical_frame" link2="gripper_l_link2" reason="Never"/>
+  <disable_collisions link1="camera_depth_optical_frame" link2="gripper_l_link_finger" reason="Never"/>
+  <disable_collisions link1="camera_depth_optical_frame" link2="gripper_tip_midpoint_arm" reason="Never"/>
+  <disable_collisions link1="camera_depth_optical_frame" link2="gripper_tip_midpoint_counterarm" reason="Never"/>
+  <disable_collisions link1="camera_depth_optical_frame" link2="gripper_tip" reason="Never"/>
+  <disable_collisions link1="camera_depth_optical_frame" link2="camera_flange_support" reason="Never"/>
+  <disable_collisions link1="camera_left_ir_frame" link2="base_link" reason="Never"/>
+  <disable_collisions link1="camera_left_ir_frame" link2="base_link_inertia" reason="Never"/>
+  <disable_collisions link1="camera_left_ir_frame" link2="shoulder_link" reason="Never"/>
+  <disable_collisions link1="camera_left_ir_frame" link2="upper_arm_link" reason="Never"/>
+  <disable_collisions link1="camera_left_ir_frame" link2="forearm_link" reason="Never"/>
+  <disable_collisions link1="camera_left_ir_frame" link2="wrist_1_link" reason="Never"/>
+  <disable_collisions link1="camera_left_ir_frame" link2="wrist_2_link" reason="Never"/>
+  <disable_collisions link1="camera_left_ir_frame" link2="wrist_3_link" reason="Never"/>
+  <disable_collisions link1="camera_left_ir_frame" link2="flange" reason="Never"/>
+  <disable_collisions link1="camera_left_ir_frame" link2="tool0" reason="Never"/>
+  <disable_collisions link1="camera_left_ir_frame" link2="gripper_base_link" reason="Never"/>
+  <disable_collisions link1="camera_left_ir_frame" link2="gripper_r_link1" reason="Never"/>
+  <disable_collisions link1="camera_left_ir_frame" link2="gripper_r_link2" reason="Never"/>
+  <disable_collisions link1="camera_left_ir_frame" link2="gripper_r_link_finger" reason="Never"/>
+  <disable_collisions link1="camera_left_ir_frame" link2="gripper_l_link1" reason="Never"/>
+  <disable_collisions link1="camera_left_ir_frame" link2="gripper_l_link2" reason="Never"/>
+  <disable_collisions link1="camera_left_ir_frame" link2="gripper_l_link_finger" reason="Never"/>
+  <disable_collisions link1="camera_left_ir_frame" link2="gripper_tip_midpoint_arm" reason="Never"/>
+  <disable_collisions link1="camera_left_ir_frame" link2="gripper_tip_midpoint_counterarm" reason="Never"/>
+  <disable_collisions link1="camera_left_ir_frame" link2="gripper_tip" reason="Never"/>
+  <disable_collisions link1="camera_left_ir_frame" link2="camera_flange_support" reason="Never"/>
+  <disable_collisions link1="camera_left_ir_optical_frame" link2="base_link" reason="Never"/>
+  <disable_collisions link1="camera_left_ir_optical_frame" link2="base_link_inertia" reason="Never"/>
+  <disable_collisions link1="camera_left_ir_optical_frame" link2="shoulder_link" reason="Never"/>
+  <disable_collisions link1="camera_left_ir_optical_frame" link2="upper_arm_link" reason="Never"/>
+  <disable_collisions link1="camera_left_ir_optical_frame" link2="forearm_link" reason="Never"/>
+  <disable_collisions link1="camera_left_ir_optical_frame" link2="wrist_1_link" reason="Never"/>
+  <disable_collisions link1="camera_left_ir_optical_frame" link2="wrist_2_link" reason="Never"/>
+  <disable_collisions link1="camera_left_ir_optical_frame" link2="wrist_3_link" reason="Never"/>
+  <disable_collisions link1="camera_left_ir_optical_frame" link2="flange" reason="Never"/>
+  <disable_collisions link1="camera_left_ir_optical_frame" link2="tool0" reason="Never"/>
+  <disable_collisions link1="camera_left_ir_optical_frame" link2="gripper_base_link" reason="Never"/>
+  <disable_collisions link1="camera_left_ir_optical_frame" link2="gripper_r_link1" reason="Never"/>
+  <disable_collisions link1="camera_left_ir_optical_frame" link2="gripper_r_link2" reason="Never"/>
+  <disable_collisions link1="camera_left_ir_optical_frame" link2="gripper_r_link_finger" reason="Never"/>
+  <disable_collisions link1="camera_left_ir_optical_frame" link2="gripper_l_link1" reason="Never"/>
+  <disable_collisions link1="camera_left_ir_optical_frame" link2="gripper_l_link2" reason="Never"/>
+  <disable_collisions link1="camera_left_ir_optical_frame" link2="gripper_l_link_finger" reason="Never"/>
+  <disable_collisions link1="camera_left_ir_optical_frame" link2="gripper_tip_midpoint_arm" reason="Never"/>
+  <disable_collisions link1="camera_left_ir_optical_frame" link2="gripper_tip_midpoint_counterarm" reason="Never"/>
+  <disable_collisions link1="camera_left_ir_optical_frame" link2="gripper_tip" reason="Never"/>
+  <disable_collisions link1="camera_left_ir_optical_frame" link2="camera_flange_support" reason="Never"/>
+  <disable_collisions link1="camera_right_ir_frame" link2="base_link" reason="Never"/>
+  <disable_collisions link1="camera_right_ir_frame" link2="base_link_inertia" reason="Never"/>
+  <disable_collisions link1="camera_right_ir_frame" link2="shoulder_link" reason="Never"/>
+  <disable_collisions link1="camera_right_ir_frame" link2="upper_arm_link" reason="Never"/>
+  <disable_collisions link1="camera_right_ir_frame" link2="forearm_link" reason="Never"/>
+  <disable_collisions link1="camera_right_ir_frame" link2="wrist_1_link" reason="Never"/>
+  <disable_collisions link1="camera_right_ir_frame" link2="wrist_2_link" reason="Never"/>
+  <disable_collisions link1="camera_right_ir_frame" link2="wrist_3_link" reason="Never"/>
+  <disable_collisions link1="camera_right_ir_frame" link2="flange" reason="Never"/>
+  <disable_collisions link1="camera_right_ir_frame" link2="tool0" reason="Never"/>
+  <disable_collisions link1="camera_right_ir_frame" link2="gripper_base_link" reason="Never"/>
+  <disable_collisions link1="camera_right_ir_frame" link2="gripper_r_link1" reason="Never"/>
+  <disable_collisions link1="camera_right_ir_frame" link2="gripper_r_link2" reason="Never"/>
+  <disable_collisions link1="camera_right_ir_frame" link2="gripper_r_link_finger" reason="Never"/>
+  <disable_collisions link1="camera_right_ir_frame" link2="gripper_l_link1" reason="Never"/>
+  <disable_collisions link1="camera_right_ir_frame" link2="gripper_l_link2" reason="Never"/>
+  <disable_collisions link1="camera_right_ir_frame" link2="gripper_l_link_finger" reason="Never"/>
+  <disable_collisions link1="camera_right_ir_frame" link2="gripper_tip_midpoint_arm" reason="Never"/>
+  <disable_collisions link1="camera_right_ir_frame" link2="gripper_tip_midpoint_counterarm" reason="Never"/>
+  <disable_collisions link1="camera_right_ir_frame" link2="gripper_tip" reason="Never"/>
+  <disable_collisions link1="camera_right_ir_frame" link2="camera_flange_support" reason="Never"/>
+  <disable_collisions link1="camera_right_ir_optical_frame" link2="base_link" reason="Never"/>
+  <disable_collisions link1="camera_right_ir_optical_frame" link2="base_link_inertia" reason="Never"/>
+  <disable_collisions link1="camera_right_ir_optical_frame" link2="shoulder_link" reason="Never"/>
+  <disable_collisions link1="camera_right_ir_optical_frame" link2="upper_arm_link" reason="Never"/>
+  <disable_collisions link1="camera_right_ir_optical_frame" link2="forearm_link" reason="Never"/>
+  <disable_collisions link1="camera_right_ir_optical_frame" link2="wrist_1_link" reason="Never"/>
+  <disable_collisions link1="camera_right_ir_optical_frame" link2="wrist_2_link" reason="Never"/>
+  <disable_collisions link1="camera_right_ir_optical_frame" link2="wrist_3_link" reason="Never"/>
+  <disable_collisions link1="camera_right_ir_optical_frame" link2="flange" reason="Never"/>
+  <disable_collisions link1="camera_right_ir_optical_frame" link2="tool0" reason="Never"/>
+  <disable_collisions link1="camera_right_ir_optical_frame" link2="gripper_base_link" reason="Never"/>
+  <disable_collisions link1="camera_right_ir_optical_frame" link2="gripper_r_link1" reason="Never"/>
+  <disable_collisions link1="camera_right_ir_optical_frame" link2="gripper_r_link2" reason="Never"/>
+  <disable_collisions link1="camera_right_ir_optical_frame" link2="gripper_r_link_finger" reason="Never"/>
+  <disable_collisions link1="camera_right_ir_optical_frame" link2="gripper_l_link1" reason="Never"/>
+  <disable_collisions link1="camera_right_ir_optical_frame" link2="gripper_l_link2" reason="Never"/>
+  <disable_collisions link1="camera_right_ir_optical_frame" link2="gripper_l_link_finger" reason="Never"/>
+  <disable_collisions link1="camera_right_ir_optical_frame" link2="gripper_tip_midpoint_arm" reason="Never"/>
+  <disable_collisions link1="camera_right_ir_optical_frame" link2="gripper_tip_midpoint_counterarm" reason="Never"/>
+  <disable_collisions link1="camera_right_ir_optical_frame" link2="gripper_tip" reason="Never"/>
+  <disable_collisions link1="camera_right_ir_optical_frame" link2="camera_flange_support" reason="Never"/>
 </robot>

Commit message: fix(bringup): SRDF home 同步现场定版 [90,-45,35,-70,-90,0]°（与 demo HOME_JOINTS 一致；之前 RViz goal-state 选 home 是老默认值，跟真机 go_home 对不上）；jetson_up --build 默认 JOBS=2（8G 全核 colcon OOM，忘带差点又炸）

File: src/ur5_bringup/srdf/ur5_with_gripper.srdf.xacro (robot description, xacro)
@@ -18,9 +18,12 @@
   </group>
   <group_state name="home" group="ur_manipulator">
-    <joint name="elbow_joint" value="0" />
+    <!-- 现场定版（2026-10-13 示教器抄录 [90,-45,35,-70,-90,0]°，与 demo 的
+         HOME_JOINTS / UR5_HOME_JOINTS 一致；dfd991e 之前这里是老默认值，
+         RViz goal-state 选 home 会跟真机 go_home 对不上） -->
+    <joint name="elbow_joint" value="0.6109" />
     <joint name="shoulder_lift_joint" value="-0.7854" />
-    <joint name="shoulder_pan_joint" value="0" />
-    <joint name="wrist_1_joint" value="0" />
-    <joint name="wrist_2_joint" value="0" />
+    <joint name="shoulder_pan_joint" value="1.5708" />
+    <joint name="wrist_1_joint" value="-1.2217" />
+    <joint name="wrist_2_joint" value="-1.5708" />
     <joint name="wrist_3_joint" value="0" />
   </group_state>

Commit message: config(home): 二定版 home [116.8,-45.8,35,-89.1,-90,0]°——真桌子挪位后手工对准桌面抄录（pan +26.8° 与桌面 30° 偏角闭环）；HOME_JOINTS 与 SRDF home 同步

File: src/ur5_bringup/srdf/ur5_with_gripper.srdf.xacro (robot description, xacro)
@@ -18,11 +18,10 @@
   </group>
   <group_state name="home" group="ur_manipulator">
-    <!-- 现场定版（2026-10-13 示教器抄录 [90,-45,35,-70,-90,0]°，与 demo 的
-         HOME_JOINTS / UR5_HOME_JOINTS 一致；dfd991e 之前这里是老默认值，
-         RViz goal-state 选 home 会跟真机 go_home 对不上） -->
+    <!-- 现场二定版（2026-10-29，桌子挪位后手工对准桌面抄录 [116.8,-45.8,35,-89.1,-90,0]°，
+         与 demo 的 HOME_JOINTS / UR5_HOME_JOINTS 一致） -->
     <joint name="elbow_joint" value="0.6109" />
-    <joint name="shoulder_lift_joint" value="-0.7854" />
-    <joint name="shoulder_pan_joint" value="1.5708" />
-    <joint name="wrist_1_joint" value="-1.2217" />
+    <joint name="shoulder_lift_joint" value="-0.7994" />
+    <joint name="shoulder_pan_joint" value="2.0375" />
+    <joint name="wrist_1_joint" value="-1.555" />
     <joint name="wrist_2_joint" value="-1.5708" />
     <joint name="wrist_3_joint" value="0" />
